Commit message: modify LIO_SAM params file

File: install/lio_sam/share/lio_sam/config/robot.urdf.xacro (robot description, xacro)
@@ -1 +1 @@
-/home/ngin/LAB/Resfes24/Robot_LiDAR3d/src/lio_sam/config/robot.urdf.xacro
+/home/ngin/LAB/Resfes24/Robot_LiDAR3d/src/LIO-SAM/config/robot.urdf.xacro

File: src/pochita/description/gazebo_control.xacro (robot description, xacro)
@@ -4,5 +4,5 @@
         <plugin name="diff_drive" filename="libgazebo_ros_diff_drive.so">
             <ros>
-                <!-- <namespace>/odometry</namespace> -->
+                <namespace>/sensor</namespace>
             </ros>
             <left_joint>left_wheel_joint</left_joint>
@@ -16,5 +16,5 @@
             <robot_base_frame>base_link</robot_base_frame>
             <publish_odom>true</publish_odom>
-            <publish_odom_tf>true</publish_odom_tf>
+            <publish_odom_tf>false</publish_odom_tf>
             <publish_wheel_tf>true</publish_wheel_tf>
         </plugin>

File: src/pochita/description/imu.xacro (robot description, xacro)
@@ -2,8 +2,9 @@
 <robot xmlns:xacro="http://www.ros.org/wiki/xacro"  name="robot">
     <xacro:include filename="inertial_macros.xacro"/>
+    <!-- <xacro:include filename="materials.xacro"/> -->
     <joint name="imu_joint" type="fixed">
-        <parent link="base_link"/>
-        <child link="imu_link"/>
-        <origin xyz="0 0 0.075"/>
+      <parent link="base_link"/>
+      <child link="imu_link"/>
+      <origin xyz="0 0 0.075"/>
     </joint>
     <link name="imu_link">
@@ -22,30 +23,10 @@
         </xacro:inertial_box>
     </link>
-    <!-- <gazebo reference="imu_link">
-      <gravity>true</gravity>
-      <sensor name="imu_sensor" type="imu">
-        <always_on>true</always_on>
-        <update_rate>100</update_rate>
-        <visualize>true</visualize>
-        <topic>__default_topic__</topic>
-        <plugin filename="libgazebo_ros_imu_sensor.so" name="imu_plugin">
-          <topicName>imu</topicName>
-          <bodyName>imu_link</bodyName>
-          <updateRateHZ>10.0</updateRateHZ>
-          <gaussianNoise>0.0</gaussianNoise>
-          <xyzOffset>0 0 0</xyzOffset>
-          <rpyOffset>0 0 0</rpyOffset>
-          <frameName>imu_link</frameName>
-          <initialOrientationAsReference>false</initialOrientationAsReference>
-        </plugin>
-        <pose>0 0 0 0 0 0</pose>
-      </sensor>
-    </gazebo>
-     -->
     <gazebo reference="imu_link">
+        <gravity>true</gravity>
         <sensor name="imu_sensor" type="imu">
          <plugin filename="libgazebo_ros_imu_sensor.so" name="imu_plugin">
             <ros>
-              <!-- <namespace>odometry</namespace> -->
+              <namespace>/sensor</namespace>
               <remapping>~/out:=imu</remapping>
             </ros>
@@ -53,5 +34,5 @@
           </plugin>
           <always_on>true</always_on>
-          <update_rate>1000</update_rate>
+          <update_rate>150</update_rate>
           <visualize>true</visualize>
           <imu>
@@ -110,23 +91,4 @@
           </imu>
         </sensor>
-    </gazebo>
-    <!-- <gazebo reference="imu_link">
-      <gravity>true</gravity>
-      <sensor name="imu_sensor" type="imu">
-        <always_on>true</always_on>
-        <update_rate>1000</update_rate>
-        <visualize>true</visualize>
-        <topic>__default_topic__</topic>
-        <plugin filename="libgazebo_ros_imu_sensor.so" name="imu_plugin">
-          <topicName>trunk_imu</topicName>
-          <bodyName>imu_link</bodyName>
-          <updateRateHZ>1000.0</updateRateHZ>
-          <gaussianNoise>0.0</gaussianNoise>
-          <xyzOffset>0 0 0</xyzOffset>
-          <rpyOffset>0 0 0</rpyOffset>
-          <frameName>imu_link</frameName>
-        </plugin>
-        <pose>0 0 0 0 0 0</pose>
-      </sensor>
-    </gazebo> -->
+  </gazebo>
 </robot>

File: src/pochita/description/robot.urdf.xacro (robot description, xacro)
@@ -3,6 +3,7 @@
     <xacro:include filename="robot_core.xacro"/>
     <xacro:include filename="gazebo_control.xacro"/>
-    <xacro:include filename="lidar.xacro"/>
+    <!-- <xacro:include filename="lidar.xacro"/> -->
+    <xacro:include filename="velodyne.xacro"/>
     <xacro:include filename="camera.xacro"/>
-    <!-- <xacro:include filename="imu.xacro"/> -->
+    <xacro:include filename="imu.xacro"/>
 </robot>

File: src/pochita/description/robot_core.xacro (robot description, xacro)
@@ -13,94 +13,4 @@
     <link name="base_footprint">
     </link>
-    <!-- IMU LINK -->
-    <joint name="imu_joint" type="fixed">
-        <parent link="base_link"/>
-        <child link="imu_link"/>
-        <origin xyz="0 0 0.075"/>
-    </joint>
-    <link name="imu_link">
-        <visual>
-          <geometry>
-            <box size="0.1 0.1 0.1"/>
-          </geometry>
-        </visual>
-        <collision>
-          <geometry>
-            <box size="0.1 0.1 0.1"/>
-          </geometry>
-        </collision>
-        <xacro:inertial_box mass="0.1" x="0.1" y="0.1" z="0.1">
-          <origin xyz="0. 0 0.0" rpy="0 0 0"/>
-        </xacro:inertial_box>
-    </link>
-    <gazebo reference="imu_link">
-        <gravity>true</gravity>
-        <sensor name="imu_sensor" type="imu">
-         <plugin filename="libgazebo_ros_imu_sensor.so" name="imu_plugin">
-            <ros>
-              <!-- <namespace>odometry</namespace> -->
-              <remapping>~/out:=imu</remapping>
-            </ros>
-            <initial_orientation_as_reference>true</initial_orientation_as_reference>
-          </plugin>
-          <always_on>true</always_on>
-          <update_rate>150</update_rate>
-          <visualize>true</visualize>
-          <imu>
-            <angular_velocity>
-              <x>
-                <noise type="gaussian">
-                  <mean>0.0</mean>
-                  <stddev>2e-4</stddev>
-                  <bias_mean>0.0000075</bias_mean>
-                  <bias_stddev>0.0000008</bias_stddev>
-                </noise>
-              </x>
-              <y>
-                <noise type="gaussian">
-                  <mean>0.0</mean>
-                  <stddev>2e-4</stddev>
-                  <bias_mean>0.0000075</bias_mean>
-                  <bias_stddev>0.0000008</bias_stddev>
-                </noise>
-              </y>
-              <z>
-                <noise type="gaussian">
-                  <mean>0.0</mean>
-                  <stddev>2e-4</stddev>
-                  <bias_mean>0.0000075</bias_mean>
-                  <bias_stddev>0.0000008</bias_stddev>
-                </noise>
-              </z>
-            </angular_velocity>
-            <linear_acceleration>
-              <x>
-                <noise type="gaussian">
-                  <mean>0.0</mean>
-                  <stddev>1.7e-2</stddev>
-                  <bias_mean>0.1</bias_mean>
-                  <bias_stddev>0.001</bias_stddev>
-                </noise>
-              </x>
-              <y>
-                <noise type="gaussian">
-                  <mean>0.0</mean>
-                  <stddev>1.7e-2</stddev>
-                  <bias_mean>0.1</bias_mean>
-                  <bias_stddev>0.001</bias_stddev>
-                </noise>
-              </y>
-              <z>
-                <noise type="gaussian">
-                  <mean>0.0</mean>
-                  <stddev>1.7e-2</stddev>
-                  <bias_mean>0.1</bias_mean>
-                  <bias_stddev>0.001</bias_stddev>
-                </noise>
-              </z>
-            </linear_acceleration>
-          </imu>
-        </sensor>
-    </gazebo>
     <!-- CHASSIS LINK -->
     <joint name="chassis_joint" type="fixed">

File: src/pochita/description/velodyne.xacro (robot description, xacro)
@@ -55,4 +55,8 @@
             </ray>
             <plugin name="velodyne" filename="libgazebo_ros_velodyne_laser.so">
+                <ros>
+                    <namespace>/sensor</namespace>
+                    <remapping>~/out:=velodyne</remapping>
+                  </ros>
                 <gaussianNoise>0.00</gaussianNoise>
                 <hokuyoMinIntensity>1</hokuyoMinIntensity>
